Commit message: tmp

File: assets/wheel_leg_car_2links/wheel_leg_car_2links.urdf (robot description, URDF)
Before this commit: robot wheel_leg_car_2links, 8 links, 7 joints
Links:
- added link gimbal_pitch_link, mass 0.25; collision box size=0.28 0.04 0.04; visual box size=0.28 0.04 0.04
- added link gimbal_yaw_link, mass 0.2775; collision box size=0.036 0.036 0.18; visual box size=0.036 0.036 0.18
Joints:
- added joint gimbal_pitch_joint: type fixed, parent gimbal_yaw_link, child gimbal_pitch_link, origin xyz=-0.09 0 0.156 rpy=0 0 0
- added joint gimbal_yaw_joint: type continuous, parent base_link, child gimbal_yaw_link, origin xyz=0 0 0.06 rpy=0 0 0, axis 0 0 1, limit effort=5 velocity=30
